Commit message: Update lidar.xacro

File: asimov_description/lidar.xacro (robot description, xacro)
@@ -18,4 +18,9 @@
     </visual>
   </link>
-  <!-- no collision? -->
+  <!-- no collision? just copied geo from visual, may need edits-->
+  <collision>
+      <geometry>
+        <box size="0.06 0.06 0.03"/>
+      </geometry>
+  </collision>
 </robot>

Commit message: Update lidar.xacro

File: asimov_description/lidar.xacro (robot description, xacro)
@@ -2,8 +2,8 @@
 <robot xmlns:xacro="http://www.ros.org/wiki/xacro" >
   <joint name="lidar_joint" type="fixed">
-        <parent link="base_link"/>
-        <child link="lidar_link"/>
-        <!-- LiDAR mounted at ? above base_link; likely needs to be edited later -->
-        <origin xyz="-0.40 -0.21 -0.01" rpy="0 0 0"/>
+    <parent link="base_link"/>
+    <child link="lidar_link"/>
+    <!-- LiDAR mounted at ? above base_link; likely needs to be edited later -->
+    <origin xyz="-0.40 -0.21 -0.01" rpy="0 0 0"/>
   </joint>
   <link name="lidar_link">

Commit message: Update lidar.xacro

File: asimov_description/lidar.xacro (robot description, xacro)
@@ -17,4 +17,12 @@
       </material>
     </visual>
+    <!-- not accurate inertial. rec is 0.001 for 0.1m box of 0.6kg. This thing is about half the size and lighter.-->
+    <inertial>
+        <mass value="0.01" />
+        <origin xyz="0 0 0" rpy="0 0 0" />
+        <inertia ixx="0.00001" ixy="0.0" ixz="0.0"
+                 iyy="0.00001" iyz="0.0"
+                 izz="0.00001" />
+    </inertial>
   </link>
   <!-- no collision? just copied geo from visual, may need edits-->
