Commit message: Update ros2_control.xacro

File: asimov_description/ros2_control.xacro (robot description, xacro)
@@ -6,5 +6,5 @@
               <plugin>gazebo_ros2_control/GazeboSystem</plugin>
           </hardware>
-          <joint name="left_wheel_joint">
+          <joint name="fl-wheel">
               <command_interface name="velocity">
                   <param name="min">-10</param>
@@ -14,5 +14,21 @@
               <state_interface name="velocity" />
           </joint>
-          <joint name="right_wheel_joint">
+          <joint name="rl-wheel">
+              <command_interface name="velocity">
+                  <param name="min">-10</param>
+                  <param name="max">10</param>
+              </command_interface>
+              <state_interface name="position" />
+              <state_interface name="velocity" />
+          </joint>
+          <joint name="fr-wheel">
+              <command_interface name="velocity">
+                  <param name="min">-10</param>
+                  <param name="max">10</param>
+              </command_interface>
+              <state_interface name="velocity" />
+              <state_interface name="position" />
+          </joint>
+          <joint name="rr-wheel">
               <command_interface name="velocity">
                   <param name="min">-10</param>
@@ -25,5 +41,7 @@
       <gazebo>
           <plugin filename="libgazebo_ros2_control.so" name="gazebo_ros2_control">
-              <parameters>$(find ASIMOV_FINAL_v3)/config/ros2controls_controllers.yaml</parameters>
+              <robot_param>robot_description</robot_param>
+      	      <robot_param_node>robot_state_publisher</robot_param_node>
+              <parameters>$(find asimov_nav2test)/config/ros2controls_controllers.yaml</parameters>
           </plugin>
       </gazebo>
